File: Kicad files/VFO na esp32.kicad_sch (KiCad schematic)
At the start: 42 parts, among them J1 Conn_01x02_Socket, J2 Conn_01x08_Socket, J3 Si5351A, J4 Conn_01x02_Socket, SW1 RotaryEncoder_Switch, SW2 STEP +, SW3 STEP -, SW4 Memory Channel, SW5 STORE, SW6 Brightness/Calibration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

Commit message: Dodano nowy plik README.md, poprawki w plikach projektu pcb w KICAD10.
Parts:
- R3: now not fitted
Changed lines of the file:
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@@
 		(on_board yes)
 		(in_pos_files yes)
-		(dnp no)
+		(dnp yes)
 		(property "Reference" "R3"
 			(at 190.246 110.236 0)
