File: Kicad files/VFO na esp32.kicad_sch (KiCad schematic)
At the start: 42 parts, among them J1 Conn_01x02_Socket, J2 Conn_01x08_Socket, J3 Si5351A, J4 Conn_01x02_Socket, SW1 RotaryEncoder_Switch, SW2 STEP +, SW3 STEP -, SW4 Memory Channel, SW5 STORE, SW6 Brightness/Calibration, U1 LM7805_TO220, U2 ESP32-DevKitC, U3 LM7809_TO220

Commit message: Poprawki w plikach schematu i pcb Kicada.
Parts:
- added H1, H2, H3, H4, H5, H6: MountingHole_Pad, MountingHole:MountingHole_2.7mm_M2.5_DIN965_Pad_TopBottom, symbol Mechanical:MountingHole_Pad
- R1, R2: value 2k2 -> 4k7
- R6, R7: value 5k6 -> 4k7
Connections:
- net GND: now also H1.1, H2.1, H3.1, H4.1, H5.1, H6.1
