File: Kicad files/VFO na esp32.kicad_pcb (KiCad board)
At the start: 2 copper layers, 150 x 75 mm, 50 parts, among them J1 Conn_01x02_Socket, J2 Conn_01x08_Socket, J3 Si5351A, J4 Conn_01x02_Socket, SW1 RotaryEncoder_Switch, SW2 STEP +, SW3 STEP -, SW4 Memory Channel, SW5 STORE, SW6 Brightness/Calibration, U1 LM7805_TO220, U2 ESP32-DevKitC, U3 LM7809_TO220

Commit message: Poprawki w plikach schematu i pcb Kicada.
Parts:
- removed ?: , 
- removed REF** (x6): MountingHole_2.5mm_Pad, MountingHole:MountingHole_2.5mm_Pad
- removed REF**: MountingHole_3.5mm_Pad, MountingHole:MountingHole_3.5mm_Pad
- added H1: MountingHole_Pad, MountingHole:MountingHole_2.7mm_M2.5_DIN965_Pad_TopBottom, F.Cu at (102.0, 65.3)
- added H2: MountingHole_Pad, MountingHole:MountingHole_2.7mm_M2.5_DIN965_Pad_TopBottom, F.Cu at (102.1, 130.3)
- added H3: MountingHole_Pad, MountingHole:MountingHole_2.7mm_M2.5_DIN965_Pad_TopBottom, F.Cu at (180.1, 110.7)
- added H4: MountingHole_Pad, MountingHole:MountingHole_2.7mm_M2.5_DIN965_Pad_TopBottom, F.Cu at (179.9, 130.4)
- added H5: MountingHole_Pad, MountingHole:MountingHole_2.7mm_M2.5_DIN965_Pad_TopBottom, F.Cu at (239.3, 66.0)
- added H6: MountingHole_Pad, MountingHole:MountingHole_2.7mm_M2.5_DIN965_Pad_TopBottom, F.Cu at (239.5, 129.9)
- R1, R2: value 2k2 -> 4k7
- R6, R7: value 5k6 -> 4k7
- moved D1 11.8 mm to (197.1, 75.3), turned to 90 degrees
- moved C13 4.48 mm to (207.2, 67.9), turned to -90 degrees
- moved C8 2.60 mm to (204.4, 71.4)
- moved C12 1.43 mm to (207.2, 72.0)
Routing:
- net /BTN_BAND: track 175.7 -> 181.1 mm
- net Net-(D1-A): track 8.44 -> 9.80 mm
- net +9V: track 23.6 -> 24.7 mm
- net Net-(D1-K): track 66.9 -> 67.7 mm
- net GND: vias 0 -> 69
